Commit message: orange car model urdf

File: ros2/src/launch_rviz/urdf/car.urdf (robot description, URDF)
Before this commit: robot origins, 2 links, 1 joints
Links:
- removed link base_link
- removed link right_leg
- added link car; visual box size=2.51 0.64 0.55
- added link fl; visual cylinder length=0.2 radius=0.2
- added link fr; visual cylinder length=0.2 radius=0.2
- added link rl; visual cylinder length=0.2 radius=0.2
- added link rr; visual cylinder length=0.2 radius=0.2
Joints:
- removed joint base_to_right_leg
- added joint car_to_fl: type fixed, parent car, child fl, origin xyz=0 0 0
- added joint car_to_fr: type fixed, parent car, child fr, origin xyz=0 0 0
- added joint car_to_rl: type fixed, parent car, child rl, origin xyz=0 0 0
- added joint car_to_rr: type fixed, parent car, child rr, origin xyz=0 0 0

Commit message: playing around with transforms, might delete later

File: ros2/src/launch_rviz/urdf/car.urdf (robot description, URDF)
Before this commit: robot fsds_car, 5 links, 4 joints
Joints:
- joint car_to_fl: parent car -> FSCar
- joint car_to_fr: parent car -> FSCar
- joint car_to_rl: parent car -> FSCar
- joint car_to_rr: parent car -> FSCar
